File: arduino_dummy_shield.kicad_pcb (KiCad board)
At the start: 2 copper layers, 94 x 73.7 mm, 49 parts, among them J1 Power, J10 Motor, J11 Motor, J12 Motor, J13 Motor, J14 Motor, J15 MOTOR, J16 RC, J17 RC, J18 RC, J19 RC, J2 PWM, J20 RC, J21 RC, J22 ADC, J23 Analog, J24 Analog, J25 Analog, J26 Analog, J27 Analog, J28 ADC, J29 ADC, J3 Analog, J30 CAN, J31 SPI, J32 I2C, J33 UART1, J34 UART2, J35 UART3, J36 Conn_02x16_Odd_Even, J4 PWM, J5 Analog, J6 Communication, J7 Digital, J8 ICSP, J9 RESET

Commit message: Update something
Parts:
- removed the H1 at (202.9, 105.1)
- removed the H1 at (202.9, 41.6)
- removed the H1 at (119.1, 105.1)
- removed the H1 at (119.1, 41.6)
- added H1: MountingHole, MountingHole:MountingHole_3.5mm_Pad_Via, F.Cu at (119.1, 105.1)
- added H2: MountingHole, MountingHole:MountingHole_3.5mm_Pad_Via, F.Cu at (119.1, 41.6)
- added H3: MountingHole, MountingHole:MountingHole_3.5mm_Pad_Via, F.Cu at (202.9, 41.6)
- added H4: MountingHole, MountingHole:MountingHole_3.5mm_Pad_Via, F.Cu at (202.9, 105.1)
- J10, J11, J12, J13, J14: value Motor -> MOTOR
- J23, J24, J25, J26, J27: value Analog -> ADC
- moved J8 2.54 mm to (166.0, 69.5)
- moved R2 1.28 mm to (187.5, 73.3)
- moved D3 1.27 mm to (183.8, 75.9)
- moved D2 1.27 mm to (183.8, 73.3)
- moved D1 1.27 mm to (183.8, 70.8)
- moved R1 1.27 mm to (187.4, 70.8)
- moved R3 1.27 mm to (187.4, 75.9)
Connections:
- J16 pad 1: GND -> /*8
- J16 pad 2: /*8 -> VIN
- J16 pad 3: VIN -> GND
- J17 pad 1: GND -> /*9
- J17 pad 2: /*9 -> VIN
- J17 pad 3: VIN -> GND
- J18 pad 1: GND -> /*10
- J18 pad 2: /*10 -> VIN
- J18 pad 3: VIN -> GND
- J19 pad 1: GND -> /*11
- J19 pad 2: /*11 -> VIN
- J19 pad 3: VIN -> GND
- J20 pad 1: GND -> /*12
- J20 pad 2: /*12 -> VIN
- J20 pad 3: VIN -> GND
- J21 pad 1: GND -> /*13
- J21 pad 2: /*13 -> VIN
- J21 pad 3: VIN -> GND
Routing:
- net VIN: track 100.9 -> 104.9 mm
- net /*11: track 11.9 -> 8.33 mm
- net /*12: track 12.4 -> 9.13 mm
- net +5V: track 283.2 -> 280.7 mm
- net /*10: track 13.6 -> 11.1 mm
- net /*13: track 16.2 -> 14.1 mm
- net /42: track 25.0 -> 26.8 mm
- net /*9: track 17.4 -> 15.6 mm
- net /MISO: track 11.2 -> 12.3 mm
- net /MOSI: track 8.71 -> 9.76 mm
- net /*8: track 21.6 -> 20.7 mm
- net /40: track 5.72 -> 6.24 mm
- net /36: track 5.72 -> 6.24 mm
- net /38: track 5.72 -> 6.23 mm
