File: arduino_dummy_shield.kicad_sch (KiCad schematic)
At the start: 43 parts, among them J1 Power, J10 Motor, J11 Motor, J12 Motor, J13 Motor, J14 Motor, J15 Motor, J16 RC, J17 RC, J18 RC, J19 RC, J2 PWM, J20 RC, J21 RC, J22 Analog, J23 Analog, J24 Analog, J25 Analog, J26 Analog, J27 Analog, J28 Analog, J29 Analog, J3 Analog, J30 CAN, J31 SPI, J32 I2C, J33 UART1, J34 UART2, J35 UART3, J36 Conn_02x16_Odd_Even, J4 PWM, J5 Analog, J6 Communication, J7 Digital, J8 ICSP, J9 RESET

Commit message: Update something
Parts:
- added H1, H2, H3, H4: MountingHole, MountingHole:MountingHole_3.5mm_Pad_Via, symbol Mechanical:MountingHole
- J10, J11, J12, J13, J14, J15: value Motor -> MOTOR
- J22, J23, J24, J25, J26, J27, J28, J29: value Analog -> ADC
Connections:
- net *10: now also J18.1 (Pin_1); no longer J18.2 (Pin_2)
- net *11: now also J19.1 (Pin_1); no longer J19.2 (Pin_2)
- net *12: now also J20.1 (Pin_1); no longer J20.2 (Pin_2)
- net *13: now also J21.1 (Pin_1); no longer J21.2 (Pin_2)
- net *8: now also J16.1 (Pin_1); no longer J16.2 (Pin_2)
- net *9: now also J17.1 (Pin_1); no longer J17.2 (Pin_2)
- net GND: now also J16.3 (Pin_3), J17.3 (Pin_3), J18.3 (Pin_3), J19.3 (Pin_3), J20.3 (Pin_3), J21.3 (Pin_3); no longer J16.1 (Pin_1), J17.1 (Pin_1), J18.1 (Pin_1), J19.1 (Pin_1), J20.1 (Pin_1), J21.1 (Pin_1)
- net VIN: now also J16.2 (Pin_2), J17.2 (Pin_2), J18.2 (Pin_2), J19.2 (Pin_2), J20.2 (Pin_2), J21.2 (Pin_2); no longer J16.3 (Pin_3), J17.3 (Pin_3), J18.3 (Pin_3), J19.3 (Pin_3), J20.3 (Pin_3), J21.3 (Pin_3)
Other:
- moved on the sheet: J16, J17, J18, J19, J20, J21
